Commit message: Tighter FOAM collision model with chassis collision sub-links
Regenerate wheelchair_spherized.urdf with FOAM using a finer CoACD
decomposition of the chassis (24 pieces instead of 8) and per-link
sphere budgets (arm links x2, knuckles/fingers x0.5): 206 spheres. The
chassis spheres now protrude at most 174 mm (was 288 mm), and false
self-collisions over random arm poses drop from 17.8% to 10.1% versus
exact mesh checks, with no missed collisions.

- decompose_robot.sh: anchor the include pattern ('^base_link$'); a bare
  'base_link' also matched xarm_gripper_base_link and decomposed the
  gripper too.
- split_collision_link.py (run by spherize_robot.sh after FOAM): move the
  144 chassis spheres onto 12 fixed child links by spatial clustering and
  mirror base_link's SRDF disables onto them. The spheres and the
  self-collision pairs are unchanged, but each cluster gets its own tight
  bounding sphere in the generated checker, so the broad phase skips
  chassis parts the arm is nowhere near: ~1 us per configuration in a
  SIMD batch instead of ~8 us.
- Regenerate the cricket FK/collision header.

Co-Authored-By: Claude Opus 5.5 (1M context) <noreply@anthropic.com>

File: resources/robot/wheelchair/wheelchair_spherized.urdf (robot description, URDF)
Before this commit: robot wheelchair, 26 links, 25 joints
Links:
- added link base_link_collision_0; collision sphere radius=0.040324; collision sphere radius=0.040603
- added link base_link_collision_1; collision sphere radius=0.074496; collision sphere radius=0.079786
- added link base_link_collision_10; collision sphere radius=0.050054; collision sphere radius=0.050324
- added link base_link_collision_11; collision sphere radius=0.033547; collision sphere radius=0.033864
- added link base_link_collision_2; collision sphere radius=0.044776; collision sphere radius=0.048605
- added link base_link_collision_3; collision sphere radius=0.047195; collision sphere radius=0.050031
- added link base_link_collision_4; collision sphere radius=0.065146; collision sphere radius=0.065422
- added link base_link_collision_5; collision sphere radius=0.041762; collision sphere radius=0.046696
- added link base_link_collision_6; collision sphere radius=0.051346; collision sphere radius=0.058042
- added link base_link_collision_7; collision sphere radius=0.052041; collision sphere radius=0.06585
- added link base_link_collision_8; collision sphere radius=0.07799; collision sphere radius=0.080081
- added link base_link_collision_9; collision sphere radius=0.034414; collision sphere radius=0.042565
- link base_link: geometry visual mesh filename=package://meshes/base_fixed.stl
- link left_finger: geometry collision sphere radius=0.023718; collision sphere radius=0.024779
- link left_inner_knuckle: geometry collision sphere radius=0.020015; collision sphere radius=0.021056
- link left_outer_knuckle: geometry collision sphere radius=0.016872; collision sphere radius=0.0173
- link link1: geometry collision sphere radius=0.08051; collision sphere radius=0.082405
- link link2: geometry collision sphere radius=0.05706; collision sphere radius=0.059383
- link link3: geometry collision sphere radius=0.057955; collision sphere radius=0.060511
- link link4: geometry collision sphere radius=0.049704; collision sphere radius=0.052523
- link link5: geometry collision sphere radius=0.047642; collision sphere radius=0.060203
- link link6: geometry collision sphere radius=0.053225; collision sphere radius=0.053291
- link link_base: geometry collision sphere radius=0.087042; collision sphere radius=0.095256
- link right_finger: geometry collision sphere radius=0.023204; collision sphere radius=0.025204
- link right_inner_knuckle: geometry collision sphere radius=0.020151; collision sphere radius=0.020278
- link right_outer_knuckle: geometry collision sphere radius=0.017545; collision sphere radius=0.017688
- link xarm_gripper_base_link: geometry collision sphere radius=0.072277; visual mesh filename=package://meshes/base_link.stl
Joints:
- added joint base_link_collision_0_joint: type fixed, parent base_link, child base_link_collision_0, origin xyz=0 0 0 rpy=0 0 0
- added joint base_link_collision_10_joint: type fixed, parent base_link, child base_link_collision_10, origin xyz=0 0 0 rpy=0 0 0
- added joint base_link_collision_11_joint: type fixed, parent base_link, child base_link_collision_11, origin xyz=0 0 0 rpy=0 0 0
- added joint base_link_collision_1_joint: type fixed, parent base_link, child base_link_collision_1, origin xyz=0 0 0 rpy=0 0 0
- added joint base_link_collision_2_joint: type fixed, parent base_link, child base_link_collision_2, origin xyz=0 0 0 rpy=0 0 0
- added joint base_link_collision_3_joint: type fixed, parent base_link, child base_link_collision_3, origin xyz=0 0 0 rpy=0 0 0
- added joint base_link_collision_4_joint: type fixed, parent base_link, child base_link_collision_4, origin xyz=0 0 0 rpy=0 0 0
- added joint base_link_collision_5_joint: type fixed, parent base_link, child base_link_collision_5, origin xyz=0 0 0 rpy=0 0 0
- added joint base_link_collision_6_joint: type fixed, parent base_link, child base_link_collision_6, origin xyz=0 0 0 rpy=0 0 0
- added joint base_link_collision_7_joint: type fixed, parent base_link, child base_link_collision_7, origin xyz=0 0 0 rpy=0 0 0
- added joint base_link_collision_8_joint: type fixed, parent base_link, child base_link_collision_8, origin xyz=0 0 0 rpy=0 0 0
- added joint base_link_collision_9_joint: type fixed, parent base_link, child base_link_collision_9, origin xyz=0 0 0 rpy=0 0 0
