Commit message: Fix collision model: bake mesh scale to metres; regenerate spherized URDF + FK header
The wheelchair chassis/lip/wheel meshes are in millimetres (URDF
scale=0.001), but foam ignores the URDF scale during spherization, so the
chassis spheres came out 1000x too big (radius ~326 m) and every config
reported self-collision. build_robot_description.py now bakes each mesh's
scale into the geometry (copy_meshes via trimesh) and resets the URDF
scale to identity, so foam/cricket/pinocchio all see consistent metres.

Regenerated on crane0: wheelchair_spherized.urdf (95 spheres, rmax 0.33 m)
and ext/ompl_vamp/robot/wheelchair.hh (dimension=10). Verified end-to-end:
validate(HOME)=True, ~73% of sampled configs collision-free, wheelchair_arm
RRTConnect planning succeeds.

Also gitignore .scratch/ (local build scripts / logs / reference clone).

Co-Authored-By: Claude Opus 4.8 (1M context) <noreply@anthropic.com>

File: resources/robot/wheelchair/wheelchair.urdf (robot description, URDF)
Before this commit: robot wheelchair, 34 links, 33 joints
Links:
- link back_left_1: geometry collision mesh filename=package://meshes/back.stl; visual mesh filename=package://meshes/back.stl
- link back_right_1: geometry collision mesh filename=package://meshes/back.stl; visual mesh filename=package://meshes/back.stl
- link base_link: geometry collision mesh filename=package://meshes/base_fixed.stl; visual mesh filename=package://meshes/base_fixed.stl
- link front_left_1: geometry collision mesh filename=package://meshes/front.stl; visual mesh filename=package://meshes/front.stl
- link front_right_1: geometry collision mesh filename=package://meshes/front.stl; visual mesh filename=package://meshes/front.stl
- link lip_1: geometry collision mesh filename=package://meshes/lip_1.stl; visual mesh filename=package://meshes/lip_1.stl

File: resources/robot/wheelchair/wheelchair_base.urdf (robot description, URDF)
Before this commit: robot wheelchair, 38 links, 37 joints
Links:
- link back_left_1: geometry collision mesh filename=package://meshes/back.stl; visual mesh filename=package://meshes/back.stl
- link back_right_1: geometry collision mesh filename=package://meshes/back.stl; visual mesh filename=package://meshes/back.stl
- link base_link: geometry collision mesh filename=package://meshes/base_fixed.stl; visual mesh filename=package://meshes/base_fixed.stl
- link front_left_1: geometry collision mesh filename=package://meshes/front.stl; visual mesh filename=package://meshes/front.stl
- link front_right_1: geometry collision mesh filename=package://meshes/front.stl; visual mesh filename=package://meshes/front.stl
- link lip_1: geometry collision mesh filename=package://meshes/lip_1.stl; visual mesh filename=package://meshes/lip_1.stl

File: resources/robot/wheelchair/wheelchair_base_simple.urdf (robot description, URDF)
Before this commit: robot wheelchair, 26 links, 25 joints
Links:
- link back_left_1: geometry collision mesh filename=package://meshes/back.stl; visual mesh filename=package://meshes/back.stl
- link back_right_1: geometry collision mesh filename=package://meshes/back.stl; visual mesh filename=package://meshes/back.stl
- link base_link: geometry collision mesh filename=package://meshes/base_fixed.stl; visual mesh filename=package://meshes/base_fixed.stl
- link front_left_1: geometry collision mesh filename=package://meshes/front.stl; visual mesh filename=package://meshes/front.stl
- link front_right_1: geometry collision mesh filename=package://meshes/front.stl; visual mesh filename=package://meshes/front.stl

File: resources/robot/wheelchair/wheelchair_simple.urdf (robot description, URDF)
Before this commit: robot wheelchair, 22 links, 21 joints
Links:
- link back_left_1: geometry collision mesh filename=package://meshes/back.stl; visual mesh filename=package://meshes/back.stl
- link back_right_1: geometry collision mesh filename=package://meshes/back.stl; visual mesh filename=package://meshes/back.stl
- link base_link: geometry collision mesh filename=package://meshes/base_fixed.stl; visual mesh filename=package://meshes/base_fixed.stl
- link front_left_1: geometry collision mesh filename=package://meshes/front.stl; visual mesh filename=package://meshes/front.stl
- link front_right_1: geometry collision mesh filename=package://meshes/front.stl; visual mesh filename=package://meshes/front.stl

File: resources/robot/wheelchair/wheelchair_spherized.urdf (robot description, URDF)
Before this commit: robot wheelchair, 26 links, 25 joints
Links:
- link back_left_1: geometry collision sphere radius=0.125902; visual mesh filename=package://meshes/back.stl
- link back_right_1: geometry collision sphere radius=0.135849; visual mesh filename=package://meshes/back.stl
- link base_link: geometry collision sphere radius=0.109746; collision sphere radius=0.12087
- link front_left_1: geometry collision sphere radius=0.135528; collision sphere radius=0.135648
- link front_right_1: geometry collision sphere radius=0.126117; collision sphere radius=0.127501

Commit message: Add the front lip to the collision model and rebuild the planning description
The lip (lip_1) was stripped from the planning URDFs by STRIP_LINK_PREFIXES,
so it had no FOAM spheres and VAMP never checked it: whole-body plans could
drive the lip into counters and tables while reporting zero collisions
(measured: 7 cm into the RLS kitchen counter).

- build_robot_description.py: stop stripping lip_1; treat it like the frozen
  wheels (disable lip vs chassis / wheels / arm mount) so it is still checked
  against the arm and the environment.
- Regenerate the planning URDFs, SRDF, spherized URDF (6 lip spheres, 214
  total) and ext/ompl_vamp/robot/wheelchair.hh from the updated
  wheelchair_xarm_description submodule (a6d306e: new base_fixed.stl).
- CMakeLists.txt: point FindBoost at CONDA_PREFIX so a system Boost in
  /usr/include can't shadow pixi's.

wheelchair.hh was rendered with the cricket templates from 1d599b8:
`pixi run generate-fk` with the current cricket submodule (bumped in
fad2c1a) emits a header that does not compile.

Co-Authored-By: Claude Opus 5.5 <noreply@anthropic.com>

File: resources/robot/wheelchair/wheelchair.urdf (robot description, URDF)
Before this commit: robot wheelchair, 34 links, 33 joints
Links:
- removed link laser_left
- removed link laser_right
Joints:
- removed joint lidar_left_joint
- removed joint lidar_right_joint

File: resources/robot/wheelchair/wheelchair_base.urdf (robot description, URDF)
Before this commit: robot wheelchair, 38 links, 37 joints
Links:
- removed link laser_left
- removed link laser_right
Joints:
- removed joint lidar_left_joint
- removed joint lidar_right_joint

File: resources/robot/wheelchair/wheelchair_base_simple.urdf (robot description, URDF)
Before this commit: robot wheelchair, 26 links, 25 joints
Links:
- added link lip_1, mass 18.27800057815573; collision mesh filename=package://meshes/lip_1.stl; visual mesh filename=package://meshes/lip_1.stl
Joints:
- added joint Lip_joint: type fixed, parent base_link, child lip_1, origin xyz=0.58288042351 -0.135  0.14078186452388763 rpy=0 0 0

File: resources/robot/wheelchair/wheelchair_simple.urdf (robot description, URDF)
Before this commit: robot wheelchair, 22 links, 21 joints
Links:
- added link lip_1, mass 18.27800057815573; collision mesh filename=package://meshes/lip_1.stl; visual mesh filename=package://meshes/lip_1.stl
Joints:
- added joint Lip_joint: type fixed, parent base_link, child lip_1, origin xyz=0.58288042351 -0.135  0.14078186452388763 rpy=0 0 0

File: resources/robot/wheelchair/wheelchair_spherized.urdf (robot description, URDF)
Before this commit: robot wheelchair, 38 links, 37 joints
Links:
- added link lip_1, mass 18.27800057815573; collision sphere radius=0.081795; collision sphere radius=0.088674
- link base_link_collision_0: geometry collision sphere radius=0.039066; collision sphere radius=0.041715
- link base_link_collision_1: geometry collision sphere radius=0.023894; collision sphere radius=0.02509
- link base_link_collision_10: geometry collision sphere radius=0.025934; collision sphere radius=0.026168
- link base_link_collision_11: geometry collision sphere radius=0.048741; collision sphere radius=0.050291
- link base_link_collision_2: geometry collision sphere radius=0.064307; collision sphere radius=0.066635
- link base_link_collision_3: geometry collision sphere radius=0.045754; collision sphere radius=0.048421
- link base_link_collision_4: geometry collision sphere radius=0.080094; collision sphere radius=0.084116
- link base_link_collision_5: geometry collision sphere radius=0.053034; collision sphere radius=0.053803
- link base_link_collision_6: geometry collision sphere radius=0.033313; collision sphere radius=0.03332
- link base_link_collision_7: geometry collision sphere radius=0.037784; collision sphere radius=0.038137
- link base_link_collision_8: geometry collision sphere radius=0.042773; collision sphere radius=0.043139
- link base_link_collision_9: geometry collision sphere radius=0.04216; collision sphere radius=0.04524
- link link_eef: geometry collision sphere radius=0.027216; collision sphere radius=0.030252
Joints:
- added joint Lip_joint: type fixed, parent base_link, child lip_1, origin xyz=0.58288042351 -0.135  0.14078186452388763 rpy=0 0 0

Commit message: Fix generate-fk, deterministic mesh flattening, and guard against stale builds
- generate_fk.sh: restore the brace that cricket's fk_template.hh loses in
  `base_position = {{{join(...)}}}` (inja reads `{{{` as `{{` + a dropped `{`),
  the only thing stopping the current cricket's header from compiling.
  `pixi run generate-fk` now runs end to end again.
- build_robot_description.py: flatten mesh paths by source file, not basename.
  camera/realsense/{visual,collision}/d435_with_cam_stand.stl used to collapse
  into one name and filesystem order picked the survivor; same-named files now
  keep their folder in the flat name, each copied from its exact source, and
  the generated meshes/ dir is cleared first so dropped meshes don't linger.
- Regenerated the description with the fixed pipeline (spheres unchanged:
  214/214 identical) and the header with the current cricket templates.
- tests/test_compiled_robot_model.py: fail when the compiled extension's sphere
  model doesn't match wheelchair_spherized.urdf (a regenerated header without a
  rebuild left lip_1 unchecked), and assert an obstacle on lip_1, a chassis
  cluster and link_eef is a collision.

Co-Authored-By: Claude Opus 5.5 <noreply@anthropic.com>

File: resources/robot/wheelchair/wheelchair.urdf (robot description, URDF)
Before this commit: robot wheelchair, 32 links, 31 joints
Links:
- link link_eef: geometry collision mesh filename=package://meshes/camera_realsense_collision_d435_with_cam_s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; visual mesh filename=package://meshes/camera_realsense_visual_d435_with_cam_stan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

File: resources/robot/wheelchair/wheelchair_base.urdf (robot description, URDF)
Before this commit: robot wheelchair, 36 links, 35 joints
Links:
- link link_eef: geometry collision mesh filename=package://meshes/camera_realsense_collision_d435_with_cam_s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; visual mesh filename=package://meshes/camera_realsense_visual_d435_with_cam_stan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

File: resources/robot/wheelchair/wheelchair_base_simple.urdf (robot description, URDF)
Before this commit: robot wheelchair, 27 links, 26 joints
Links:
- link link_eef: geometry collision mesh filename=package://meshes/camera_realsense_collision_d435_with_cam_s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; visual mesh filename=package://meshes/camera_realsense_visual_d435_with_cam_stan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

File: resources/robot/wheelchair/wheelchair_simple.urdf (robot description, URDF)
Before this commit: robot wheelchair, 23 links, 22 joints
Links:
- link link_eef: geometry collision mesh filename=package://meshes/camera_realsense_collision_d435_with_cam_s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; visual mesh filename=package://meshes/camera_realsense_visual_d435_with_cam_stan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

File: resources/robot/wheelchair/wheelchair_spherized.urdf (robot description, URDF)
Before this commit: robot wheelchair, 39 links, 38 joints
Links:
- link link_eef: geometry collision sphere radius=0.027216; collision sphere radius=0.030252
